File: My Projects.kicad_sch (KiCad schematic)
At the start: 44 parts, among them IC1 7483, IC2 7483, IC3 7486, IC4 7486, SW1 SW_SPST, SW2 SW_SPST, SW3 SW_SPST, SW4 SW_SPST, SW5 SW_SPST, SW6 SW_SPST, SW7 SW_SPST, SW8 SW_SPST

Commit message: COMMIT
Parts:
- added D17, D18, D19, D20, D21, D22, D23, D24: LED, symbol Device:LED
- added R17, R18, R19, R20, R21, R22, R23, R24: R, symbol Device:R
- added SW10, SW11, SW12, SW13, SW14, SW15, SW16, SW9: SW_SPST, symbol Switch:SW_SPST
Connections:
- net A0: now also D24.2 (A)
- net A1: now also D23.2 (A)
- net A2: now also D22.2 (A)
- net A3: now also D21.2 (A)
- net A4: now also D20.2 (A)
- net A5: now also D19.2 (A)
- net A6: now also D18.2 (A)
- net A7: now also D17.2 (A)
- net GND: now also D10.1 (K), D11.1 (K), D12.1 (K), D13.1 (K), D14.1 (K), D15.1 (K), D16.1 (K), D9.1 (K), SW10.2 (B), SW11.2 (B), SW12.2 (B), SW13.2 (B), SW14.2 (B), SW15.2 (B), SW16.2 (B), SW9.2 (B)
- new net: D23.1 (K), R23.2
- new net: R24.1, SW16.1 (A)
- new net: D24.1 (K), R24.2
- new net: R18.1, SW10.1 (A)
- new net: R20.1, SW12.1 (A)
- new net: D20.1 (K), R20.2
- new net: D18.1 (K), R18.2
- new net: D17.1 (K), R17.2
- new net: R21.1, SW13.1 (A)
- new net: D21.1 (K), R21.2
- new net: R17.1, SW9.1 (A)
- new net: R19.1, SW11.1 (A)
- new net: D19.1 (K), R19.2
- new net: R23.1, SW15.1 (A)
- new net: D22.1 (K), R22.2
- new net: R22.1, SW14.1 (A)
